Commit message: connec the publish

File: steerbot/urdf/steerbot_origin.xacro (robot description, xacro)
@@ -2,12 +2,12 @@
 <robot name="steerbot" xmlns:xacro="http://www.ros.org/wiki/xacro">
     <xacro:include filename="$(find steerbot)/urdf/steerbot.specs" />
-    <xacro:include filename="$(find steerbot)/urdf/steerbot.gazebo"/>
-    <link name="base_footprint"/>
-    <joint name="base_footprint_joint" type="fixed">
+    <xacro:include filename="$(find steerbot)/urdf/steerbot_origin.gazebo"/>
+    <link name="steerbot_footprint"/>
+    <joint name="steerbot_footprint_joint" type="fixed">
         <origin xyz="0 0 0" rpy="0 0 0" />
-        <parent link="base_footprint"/>
-        <child link="base_link"/>
-    </joint>
-    <link name="base_link">
+        <parent link="steerbot_footprint"/>
+        <child link="steerbot_chassis"/>
+    </joint>
+    <link name="steerbot_chassis">
         <pose> 0 0 0 0 0 0</pose>
         <inertial>
@@ -52,7 +52,7 @@
         </inertial>
         <visual>
-            <origin xyz="0 0 0" rpy="0 0 0"/>
-            <geometry>
-                <mesh filename="package://steerbot/urdf/wheels/left_tire.stl" scale="0.001 0.001 0.001"/>
+            <origin xyz="0 0 0" rpy="0 1.5707 1.5707"/>
+            <geometry>
+                <cylinder radius="${wheel_rad}" length="${wheel_wid}"/>
             </geometry>
         </visual>
@@ -76,7 +76,7 @@
         </inertial>
         <visual>
-            <origin xyz="0 0 0" rpy="0 0 0"/>
-            <geometry>
-                <mesh filename="package://steerbot/urdf/wheels/right_tire.stl" scale="0.001 0.001 0.001"/>
+            <origin xyz="0 0 0" rpy="0 1.5707 1.5707"/>
+            <geometry>
+                <cylinder radius="${wheel_rad}" length="${wheel_wid}"/>
             </geometry>
         </visual>
@@ -147,5 +147,5 @@
         <origin xyz='${wheel_base/2.0} ${chassis_wid/2.0+wheel_rad/3.0} 0' rpy="0 0 0"/>
         <child link="front_left_strut"/>
-        <parent link="base_link"/>
+        <parent link="steerbot_chassis"/>
         <axis xyz="0 0 1" rpy="0 0 0"/>
         <limit effort="1000" velocity="1000"/>
@@ -168,5 +168,5 @@
         <origin xyz='${wheel_base/2.0} -${chassis_wid/2.0+wheel_rad/3.0} 0' rpy="0 0 0"/>
         <child link="front_right_strut"/>
-        <parent link="base_link"/>
+        <parent link="steerbot_chassis"/>
         <axis xyz="0 0 1" rpy="0 0 0"/>
         <limit effort="1000" velocity="1000"/>
@@ -192,7 +192,7 @@
         </inertial>
         <visual>
-            <origin xyz="0 0 0" rpy="0 0 0"/>
-            <geometry>
-                <mesh filename="package://steerbot/urdf/wheels/left_tire.stl" scale="0.001 0.001 0.001"/>
+            <origin xyz="0 0 0" rpy="0 1.5707 1.5707"/>
+            <geometry>
+                <cylinder radius="${wheel_rad}" length="${wheel_wid}"/>
             </geometry>
         </visual>
@@ -215,8 +215,8 @@
                 />
         </inertial>
-         <visual>
-            <origin xyz="0 0 0" rpy="0 0 0"/>
-            <geometry>
-                <mesh filename="package://steerbot/urdf/wheels/right_tire.stl" scale="0.001 0.001 0.001"/>
+        <visual>
+            <origin xyz="0 0 0" rpy="0 1.5707 1.5707"/>
+            <geometry>
+                <cylinder radius="${wheel_rad}" length="${wheel_wid}"/>
             </geometry>
         </visual>
@@ -287,5 +287,5 @@
         <origin xyz='-${wheel_base/2.0} ${chassis_wid/2.0+wheel_rad/3.0} 0' rpy="0 0 0"/>
         <child link="rear_left_strut"/>
-        <parent link="base_link"/>
+        <parent link="steerbot_chassis"/>
         <axis xyz="0 0 1" rpy="0 0 0"/>
         <limit effort="1000" velocity="1000"/>
@@ -308,38 +308,8 @@
         <origin xyz='-${wheel_base/2.0} -${chassis_wid/2.0+wheel_rad/3.0} 0' rpy="0 0 0"/>
         <child link="rear_right_strut"/>
-        <parent link="base_link"/>
+        <parent link="steerbot_chassis"/>
         <axis xyz="0 0 1" rpy="0 0 0"/>
         <limit effort="1000" velocity="1000"/>
         <dynamics damping="${bearing_damping}" friction="${bearing_friction}"/>
     </joint>
- <!--
-        insert part
-    -->
-<joint name="scan_joint" type="fixed">
-    <parent link="base_link"/>
-    <child link="base_scan"/>
-    <origin xyz="0 0 0.05" rpy="0 0 0"/>
-</joint>
-<link name="base_scan">
-    <!--<visual>
-      <origin xyz="0 +0.08 -0.04" rpy="+1.57 0 0"/>
-      <geometry>
-        <mesh filename="package://steerbot/urdf/rplidar-a2m4-r1.stl" scale="0.001 0.001 0.001"/>
-      </geometry>
-      <material name="dark"/>
-    </visual> -->
-    <collision>
-      <origin xyz="0.0 0 0.0" rpy="0 0 0"/>
-      <geometry>
-        <cylinder length="0.0315" radius="0.055"/>
-      </geometry>
-    </collision>
-    <inertial>
-      <mass value="0.114" />
-      <origin xyz="0 0 0" />
-      <inertia ixx="0.001" ixy="0.0" ixz="0.0"
-               iyy="0.001" iyz="0.0"
-               izz="0.001" />
-    </inertial>
-  </link>
 </robot>
