Commit message: divide launch

File: steerbot/urdf/steerbot.xacro (robot description, xacro)
@@ -313,5 +313,5 @@
         <dynamics damping="${bearing_damping}" friction="${bearing_friction}"/>
     </joint>
-    <!--
+ <!--
         insert part
     -->
@@ -319,5 +319,5 @@
     <parent link="steerbot_chassis"/>
     <child link="base_scan"/>
-    <origin xyz="-0.064 0 0.122" rpy="0 0 0"/>
+    <origin xyz="0 0 0.05" rpy="0 0 0"/>
 </joint>
 <link name="base_scan">
@@ -330,5 +330,5 @@
     </visual>
     <collision>
-      <origin xyz="0.015 0 chassis_hgt" rpy="0 0 0"/>
+      <origin xyz="0.0 0 0.0" rpy="0 0 0"/>
       <geometry>
         <cylinder length="0.0315" radius="0.055"/>

Commit message: lidar insert

File: steerbot/urdf/steerbot.xacro (robot description, xacro)
@@ -52,7 +52,7 @@
         </inertial>
         <visual>
-            <origin xyz="0 0 0" rpy="0 1.5707 1.5707"/>
-            <geometry>
-                <cylinder radius="${wheel_rad}" length="${wheel_wid}"/>
+            <origin xyz="0 0 0" rpy="0 0 0"/>
+            <geometry>
+                <mesh filename="package://steerbot/urdf/wheels/left_tire.stl" scale="0.001 0.001 0.001"/>
             </geometry>
         </visual>
@@ -76,7 +76,7 @@
         </inertial>
         <visual>
-            <origin xyz="0 0 0" rpy="0 1.5707 1.5707"/>
-            <geometry>
-                <cylinder radius="${wheel_rad}" length="${wheel_wid}"/>
+            <origin xyz="0 0 0" rpy="0 0 0"/>
+            <geometry>
+                <mesh filename="package://steerbot/urdf/wheels/right_tire.stl" scale="0.001 0.001 0.001"/>
             </geometry>
         </visual>
@@ -192,7 +192,7 @@
         </inertial>
         <visual>
-            <origin xyz="0 0 0" rpy="0 1.5707 1.5707"/>
-            <geometry>
-                <cylinder radius="${wheel_rad}" length="${wheel_wid}"/>
+            <origin xyz="0 0 0" rpy="0 0 0"/>
+            <geometry>
+                <mesh filename="package://steerbot/urdf/wheels/left_tire.stl" scale="0.001 0.001 0.001"/>
             </geometry>
         </visual>
@@ -215,8 +215,8 @@
                 />
         </inertial>
-        <visual>
-            <origin xyz="0 0 0" rpy="0 1.5707 1.5707"/>
-            <geometry>
-                <cylinder radius="${wheel_rad}" length="${wheel_wid}"/>
+         <visual>
+            <origin xyz="0 0 0" rpy="0 0 0"/>
+            <geometry>
+                <mesh filename="package://steerbot/urdf/wheels/right_tire.stl" scale="0.001 0.001 0.001"/>
             </geometry>
         </visual>
@@ -323,7 +323,7 @@
 <link name="base_scan">
     <visual>
-      <origin xyz="0 0 0.0" rpy="0 0 0"/>
+      <origin xyz="0 +0.08 -0.04" rpy="+1.57 0 0"/>
       <geometry>
-        <mesh filename="package://turtlebot3_description/meshes/sensors/lds.stl" scale="0.001 0.001 0.001"/>
+        <mesh filename="package://steerbot/urdf/rplidar-a2m4-r1.stl" scale="0.001 0.001 0.001"/>
       </geometry>
       <material name="dark"/>

Commit message: add the odom and map

File: steerbot/urdf/steerbot.xacro (robot description, xacro)
@@ -322,5 +322,5 @@
 </joint>
 <link name="base_scan">
-    <!--<visual>
+    <visual>
       <origin xyz="0 +0.08 -0.04" rpy="+1.57 0 0"/>
       <geometry>
@@ -328,5 +328,5 @@
       </geometry>
       <material name="dark"/>
-    </visual> -->
+    </visual>
     <collision>
       <origin xyz="0.0 0 0.0" rpy="0 0 0"/>
